Commit message: flipping lidar (180 degrees) in urdf and sdf

File: app/nav2_ws/src/navigation2/nav2_bringup/urdf/sentry_robot.urdf (robot description, URDF)
Before this commit: robot sentry_robot, 7 links, 6 joints
Joints:
- joint lidar_joint: origin xyz=0 0 0.45 rpy=0 0 0 -> xyz=0 0 0.45 rpy=3.14159 0 0
